Commit message: added kinetic to the simulation

File: penguin_description/urdf/penguin.urdf (robot description, URDF)
Before this commit: robot penguin, 7 links, 6 joints
Links:
- added link kinect_link, mass 0.564; collision box size=0.07271 0.27794 0.073; visual mesh filename=package://penguin_description/models/meshes/kinect.dae
- link upper_base_link: mass None -> 1.51143; geometry collision mesh filename=package://penguin_description/models/meshes/upper_base.dae; visual mesh filename=package://penguin_description/models/meshes/upper_base.dae
Joints:
- added joint kinect_base_joint: type fixed, parent base_link, child kinect_link, origin xyz=0.0 0.0 0.2 rpy=0.0 0.0 0.0

Commit message: fixed a problem in collision
the collision forms in the wheels were wrong .I changed them to the meshes .Also lifted the caster wheels a bit for better performance

File: penguin_description/urdf/penguin.urdf (robot description, URDF)
Before this commit: robot penguin, 8 links, 7 joints
Links:
- link LW_link: geometry collision mesh filename=package://penguin_description/models/meshes/wheels.dae; visual mesh filename=package://penguin_description/models/meshes/wheels.dae
- link RW_link: geometry collision mesh filename=package://penguin_description/models/meshes/wheels.dae; visual mesh filename=package://penguin_description/models/meshes/wheels.dae
Joints:
- joint DCW_base_joint: origin xyz=0.0 -0.085 0.0 rpy=0.0 0.0 0.0 -> xyz=0.0 -0.085 0.001 rpy=0.0 0.0 0.0
- joint TCW_base_joint: origin xyz=0.0 0.092 0.0 rpy=0.0 0.0 0.0 -> xyz=0.0 0.092 0.001 rpy=0.0 0.0 0.0

Commit message: fixed a problem with the orientation of the kinetic camera

File: penguin_description/urdf/penguin.urdf (robot description, URDF)
Before this commit: robot penguin, 8 links, 7 joints
Links:
- added link camera_depth_frame
- added link camera_depth_optical_frame
- added link camera_rgb_frame
- added link camera_rgb_optical_frame
Joints:
- added joint camera_depth_joint: type fixed, parent camera_rgb_frame, child camera_depth_frame, origin xyz=0 0.0 0 rpy=0 0 0
- added joint camera_depth_optical_joint: type fixed, parent camera_depth_frame, child camera_depth_optical_frame, origin xyz=0 0 0 rpy=0 0 -1.57079632679
- added joint camera_rgb_joint: type fixed, parent base_link, child camera_rgb_frame, origin xyz=0 0 0 rpy=0 0 -1.5707
- added joint camera_rgb_optical_joint: type fixed, parent camera_rgb_frame, child camera_rgb_optical_frame, origin xyz=0 0 0 rpy=0 0 -1.57079632679
- joint kinect_base_joint: parent base_link -> camera_rgb_frame

Commit message: fixed a problem where the wheels tf were not published so i had added a config yaml that published tf info

File: penguin_description/urdf/penguin.urdf (robot description, URDF)
Before this commit: robot penguin, 12 links, 11 joints
Links:
- removed link dummy_link
- added link base_footprint
Joints:
- removed joint dummy_joint
- added joint base_footprint_joint: type fixed, parent base_footprint, child base_link, origin xyz=0.0 0.0 0.0 rpy=0.0 0.0 0.0
- joint LW_base_joint: limit (none) -> effort=100 velocity=100
- joint RW_base_joint: limit (none) -> effort=100 velocity=100

Commit message: improved the performance but more work eeds to be done

File: penguin_description/urdf/penguin.urdf (robot description, URDF)
Before this commit: robot penguin, 12 links, 11 joints
Links:
- link DCW_link: geometry collision sphere radius=0.01; visual mesh filename=package://penguin_description/models/meshes/caster_wheels.d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
- link TCW_link: geometry collision sphere radius=0.01; visual mesh filename=package://penguin_description/models/meshes/caster_wheels.d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
Joints:
- joint DCW_base_joint: origin xyz=0.0 -0.085 0.001 rpy=0.0 0.0 0.0 -> xyz=0.0 -0.085 0.0001 rpy=0.0 0.0 0.0
- joint TCW_base_joint: origin xyz=0.0 0.092 0.001 rpy=0.0 0.0 0.0 -> xyz=0.0 0.092 0.0001 rpy=0.0 0.0 0.0
- joint camera_rgb_joint: origin xyz=0 0 0 rpy=0 0 -1.5707 -> xyz=0 0 0 rpy=0 0 0
- joint kinect_base_joint: origin xyz=0.0 0.0 0.2 rpy=0.0 0.0 0.0 -> xyz=0.0 0.0 0.2 rpy=0.0 0.0 -1.57079632679

Commit message: fixed a problem with the robot where it was sliding

File: penguin_description/urdf/penguin.urdf (robot description, URDF)
Before this commit: robot penguin, 12 links, 11 joints
Links:
- link base_link: geometry collision mesh filename=package://penguin_description/models/meshes/base.dae; visual mesh filename=package://penguin_description/models/meshes/base.dae
Joints:
- joint DCW_base_joint: origin xyz=0.0 -0.085 0.0001 rpy=0.0 0.0 0.0 -> xyz=0.085 0.0  0.000 rpy=0.0 0.0 1.57079632679
- joint LW_base_joint: origin xyz=0.08 0.003 0.0315 rpy=0.0 0.0 1.5707 -> xyz=-0.004 0.08  0.0314 rpy=0.0 0.0 3.1404
- joint RW_base_joint: origin xyz=-0.08 0.003 0.0315 rpy=0.0 0.0 -1.5707 -> xyz=-0.004 -0.08  0.0314 rpy=0.0 0.0 0.0
- joint TCW_base_joint: origin xyz=0.0 0.092 0.0001 rpy=0.0 0.0 0.0 -> xyz=-0.092 0.0  0.000 rpy=0.0 0.0 1.57079632679
- joint camera_depth_optical_joint: origin xyz=0 0 0 rpy=0 0 -1.57079632679 -> xyz=0 0 0 rpy=0 0 0.0
- joint camera_rgb_optical_joint: origin xyz=0 0 0 rpy=0 0 -1.57079632679 -> xyz=0 0 0 rpy=0 0 0.0
- joint kinect_base_joint: origin xyz=0.0 0.0 0.2 rpy=0.0 0.0 -1.57079632679 -> xyz=0.0 0.0 0.2 rpy=0.0 0.0 0.0
- joint upper_base_joint: origin xyz=0.0 0.004 0.005 rpy=0.0 0.0 0.0 -> xyz=-0.004 0.0  0.005 rpy=0.0 0.0 1.57079632679

Commit message: added imu to the robot description

File: penguin_description/urdf/penguin.urdf (robot description, URDF)
Before this commit: robot penguin, 12 links, 11 joints
Links:
- added link imu_link
Joints:
- added joint base_imu_joint: type fixed, parent base_link, child imu_link, origin xyz=0.0 0.0 0.0 rpy=0.0 0.0 0.0

Commit message: improving the kalman filter the results are better but there is slight deviation

File: penguin_description/urdf/penguin.urdf (robot description, URDF)
Before this commit: robot penguin, 13 links, 12 joints
Links:
- link imu_link: mass None -> 0.001
Joints:
- joint base_imu_joint: axis (none) -> 0 1 0

Commit message: rtab implementation

File: penguin_description/urdf/penguin.urdf (robot description, URDF)
Before this commit: robot penguin, 13 links, 12 joints
Joints:
- joint camera_depth_optical_joint: origin xyz=0 0 0 rpy=0 0 0.0 -> xyz=0 0 0 rpy=0 0 0

Commit message: fixing issues with rtab

File: penguin_description/urdf/penguin.urdf (robot description, URDF)
Before this commit: robot penguin, 13 links, 12 joints
Joints:
- joint camera_depth_optical_joint: origin xyz=0 0 0 rpy=0 0 0 -> xyz=0 0 0 rpy=-1.5707 0 -1.5707
- joint camera_rgb_optical_joint: origin xyz=0 0 0 rpy=0 0 0.0 -> xyz=0 0 0 rpy=-1.5707 0 -1.5707
