Commit message: Modify Urdf file
changing colors and adding button to chassis

File: drsina_description/urdf/drsina.urdf (robot description, URDF)
Before this commit: robot DrSina, 15 links, 14 joints
Links:
- added link emergencyButton_link; visual mesh filename=package://drsina_description/models/meshes/emergencyButton.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
- added link greenButton_link; visual mesh filename=package://drsina_description/models/meshes/buttongreen.dae
- added link lidar_link; visual mesh filename=package://drsina_description/models/meshes/lidar.dae
- added link redButton_link; visual mesh filename=package://drsina_description/models/meshes/buttonred.dae
- added link redligthL_link; visual mesh filename=package://drsina_description/models/meshes/lightbackRed.dae
- added link redligthR_link; visual mesh filename=package://drsina_description/models/meshes/lightbackRed.dae
- added link yellowligthL_link; visual mesh filename=package://drsina_description/models/meshes/lightback.dae
- added link yellowligthR_link; visual mesh filename=package://drsina_description/models/meshes/lightback.dae
Joints:
- added joint emergencyButton_joint: type fixed, parent base_link, child emergencyButton_link, origin xyz=0 0 0 rpy=0 0 0
- added joint greenButton_joint: type fixed, parent base_link, child greenButton_link, origin xyz=0 0 0 rpy=0 0 0
- added joint lidar_joint: type fixed, parent base_link, child lidar_link, origin xyz=0 0 0 rpy=0 0 0
- added joint redButton_joint: type fixed, parent base_link, child redButton_link, origin xyz=0 0 0 rpy=0 0 0
- added joint redligthL_joint: type fixed, parent base_link, child redligthL_link, origin xyz=0 0 0 rpy=0 0 0
- added joint redligthR_joint: type fixed, parent base_link, child redligthR_link, origin xyz=0 0 0 rpy=0 0 0
- added joint yellowligthL_joint: type fixed, parent base_link, child yellowligthL_link, origin xyz=0 0 0 rpy=0 0 0
- added joint yellowligthR_joint: type fixed, parent base_link, child yellowligthR_link, origin xyz=0 0 0 rpy=0 0 0

Commit message: urdf with inertial

File: drsina_description/urdf/drsina.urdf (robot description, URDF)
Before this commit: robot DrSina, 15 links, 14 joints
Links:
- added link base_footprint
- added link emergencyButton_link, mass 0.024; collision mesh filename=package://drsina_description/models/meshes/emergencyButton.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; visual mesh filename=package://drsina_description/models/meshes/emergencyButton.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
- added link greenButton_link, mass 0.009; collision mesh filename=package://drsina_description/models/meshes/buttongreen.dae; visual mesh filename=package://drsina_description/models/meshes/buttongreen.dae
- added link lidar_link, mass 0.073; collision mesh filename=package://drsina_description/models/meshes/lidar.dae; visual mesh filename=package://drsina_description/models/meshes/lidar.dae
- added link redButton_link, mass 0.009; collision mesh filename=package://drsina_description/models/meshes/buttonred.dae; visual mesh filename=package://drsina_description/models/meshes/buttonred.dae
- added link redligthL_link, mass 0.013; collision mesh filename=package://drsina_description/models/meshes/lightbackRed.dae; visual mesh filename=package://drsina_description/models/meshes/lightbackRed.dae
- added link redligthR_link, mass 0.013; collision mesh filename=package://drsina_description/models/meshes/lightbackRed.dae; visual mesh filename=package://drsina_description/models/meshes/lightbackRed.dae
- added link yellowligthL_link, mass 0.013; collision mesh filename=package://drsina_description/models/meshes/lightback.dae; visual mesh filename=package://drsina_description/models/meshes/lightback.dae
- added link yellowligthR_link, mass 0.013; collision mesh filename=package://drsina_description/models/meshes/lightback.dae; visual mesh filename=package://drsina_description/models/meshes/lightback.dae
- link LBcastlewheel_link: mass None -> 0.12357
- link LFcastlewheel_link: mass None -> 0.12357
- link Lwheel_link: mass None -> 0.58215
- link RBcastlewheel_link: mass None -> 0.12357
- link RFcastlewheel_link: mass None -> 0.12357
- link Rwheel_link: mass None -> 0.58215
- link base_link: mass None -> 28.798
- link castlewheel_wheelLBlink: mass None -> 0.194
- link castlewheel_wheelLFlink: mass None -> 0.194
- link castlewheel_wheelRBlink: mass None -> 0.194
- link castlewheel_wheelRFlink: mass None -> 0.194
- link middlecastlewheelLB_link: mass None -> 0.37662
- link middlecastlewheelLF_link: mass None -> 0.37662
- link middlecastlewheelRB_link: mass None -> 0.37662
- link middlecastlewheelRF_link: mass None -> 0.37662
Joints:
- added joint emergencyButton_joint: type fixed, parent base_link, child emergencyButton_link, origin xyz=0 0 0 rpy=0 0 0
- added joint greenButton_joint: type fixed, parent base_link, child greenButton_link, origin xyz=0 0 0 rpy=0 0 0
- added joint joint_name: type fixed, parent base_footprint, child base_link, origin xyz=0.0 0.0 0.0 rpy=0.0 0.0 0.0
- added joint lidar_joint: type fixed, parent base_link, child lidar_link, origin xyz=0 0 0 rpy=0 0 0
- added joint redButton_joint: type fixed, parent base_link, child redButton_link, origin xyz=0 0 0 rpy=0 0 0
- added joint redligthL_joint: type fixed, parent base_link, child redligthL_link, origin xyz=0 0 0 rpy=0 0 0
- added joint redligthR_joint: type fixed, parent base_link, child redligthR_link, origin xyz=0 0 0 rpy=0 0 0
- added joint yellowligthL_joint: type fixed, parent base_link, child yellowligthL_link, origin xyz=0 0 0 rpy=0 0 0
- added joint yellowligthR_joint: type fixed, parent base_link, child yellowligthR_link, origin xyz=0 0 0 rpy=0 0 0

Commit message: Adding laser scan to URDF and gazebo
Laser lidar / laser ultarsonic sensors back right and left

File: drsina_description/urdf/drsina.urdf (robot description, URDF)
Before this commit: robot DrSina, 24 links, 23 joints
Links:
- added link ultrasonic_sensor_back1, mass 0.053; collision box size=0.043 0.02 0.015; visual box size=0.043 0.02 0.015
- added link ultrasonic_sensor_left1, mass 0.053; collision box size=0.043 0.02 0.015; visual box size=0.043 0.02 0.015
- added link ultrasonic_sensor_right1, mass 0.053; collision box size=0.043 0.02 0.015; visual box size=0.043 0.02 0.015
Joints:
- added joint ultrasonic_sensor_back1_joint: type fixed, parent base_link, child ultrasonic_sensor_back1, origin xyz=-0.345 0 0.05 rpy=0 0 3.142
- added joint ultrasonic_sensor_left1_joint: type fixed, parent base_link, child ultrasonic_sensor_left1, origin xyz=0.005 -0.290 0.0 rpy=0 0 -1.570796
- added joint ultrasonic_sensor_right1_joint: type fixed, parent base_link, child ultrasonic_sensor_right1, origin xyz=0.005 0.290 0.0 rpy=0 0 1.570796
- joint lidar_joint: origin xyz=0 0 0 rpy=0 0 0 -> xyz=0.303 -0.006 0.1 rpy=0 0 0

Commit message: made the robot as stable as possible (need more work)

File: drsina_description/urdf/drsina.urdf (robot description, URDF)
Before this commit: robot DrSina, 24 links, 23 joints
Links:
- link LBcastlewheel_link: geometry collision box size=0.085 0.105 0.004; visual mesh filename=package://drsina_description/models/meshes/topcastlewheel.d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
- link LFcastlewheel_link: geometry collision box size=0.085 0.105 0.004; visual mesh filename=package://drsina_description/models/meshes/topcastlewheel.d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
- link Lwheel_link: geometry collision cylinder length=0.03 radius=0.075; visual mesh filename=package://drsina_description/models/meshes/robotwheel.dae
- link RBcastlewheel_link: geometry collision box size=0.085 0.105 0.004; visual mesh filename=package://drsina_description/models/meshes/topcastlewheel.d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
- link RFcastlewheel_link: geometry collision box size=0.085 0.105 0.004; visual mesh filename=package://drsina_description/models/meshes/topcastlewheel.d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
- link Rwheel_link: geometry collision cylinder length=0.03 radius=0.075; visual mesh filename=package://drsina_description/models/meshes/robotwheel.dae
- link castlewheel_wheelLBlink: geometry collision cylinder length=0.035 radius=0.05; visual mesh filename=package://drsina_description/models/meshes/castlewheel.dae
- link castlewheel_wheelLFlink: geometry collision cylinder length=0.035 radius=0.05; visual mesh filename=package://drsina_description/models/meshes/castlewheel.dae
- link castlewheel_wheelRBlink: geometry collision cylinder length=0.035 radius=0.05; visual mesh filename=package://drsina_description/models/meshes/castlewheel.dae
- link castlewheel_wheelRFlink: geometry collision cylinder length=0.035 radius=0.05; visual mesh filename=package://drsina_description/models/meshes/castlewheel.dae
Joints:
- joint roll_jointL: limit effort=100 velocity=100 -> effort=100 velocity=1; origin xyz=-0.0019 0.235 -0.0239 rpy=0 0 0 -> xyz=-0.0019 0.235 -0.0238 rpy=0 0 0
- joint roll_jointR: limit effort=100 velocity=100 -> effort=100 velocity=1; origin xyz=-0.0019 -0.235 -0.0239 rpy=0 0 0 -> xyz=-0.0019 -0.235 -0.0238 rpy=0 0 0
- joint roll_jointcastlewheelLB: limit effort=100 velocity=100 -> effort=1000 velocity=1
- joint roll_jointcastlewheelLF: limit effort=100 velocity=100 -> effort=1000 velocity=1
- joint roll_jointcastlewheelRB: limit effort=100 velocity=100 -> effort=1000 velocity=1
- joint roll_jointcastlewheelRF: limit effort=100 velocity=100 -> effort=1000 velocity=1
- joint roll_jointmiddlecastleLB: limit effort=100 velocity=100 -> effort=1000 velocity=1
- joint roll_jointmiddlecastleLF: limit effort=100 velocity=100 -> effort=1000 velocity=1
- joint roll_jointmiddlecastleRB: limit effort=100 velocity=100 -> effort=1000 velocity=1
- joint roll_jointmiddlecastleRF: limit effort=100 velocity=100 -> effort=1000 velocity=1

Commit message: URDF modify
Lidar / collision simplification /  chassis new / button simple etc ..

File: drsina_description/urdf/drsina.urdf (robot description, URDF)
Before this commit: robot DrSina, 23 links, 22 joints
Links:
- added link base_footprint
- added link emergencyButton2_link, mass 0.024; collision cylinder length=0.007 radius=0.025; visual cylinder length=0.007 radius=0.025
- added link ultrasonic_sensor_back1, mass 0.053; collision box size=0.043 0.02 0.015; visual box size=0.043 0.02 0.015
- added link ultrasonic_sensor_left1, mass 0.053; collision box size=0.043 0.02 0.015; visual box size=0.043 0.02 0.015
- added link ultrasonic_sensor_right1, mass 0.053; collision box size=0.043 0.02 0.015; visual box size=0.043 0.02 0.015
- link LBcastlewheel_link: mass None -> 0.12357; geometry collision mesh filename=package://drsina_description/models/meshes/topcastlewheel.d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; visual mesh filename=package://drsina_description/models/meshes/topcastlewheel.d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
- link LFcastlewheel_link: mass None -> 0.12357; geometry collision mesh filename=package://drsina_description/models/meshes/topcastlewheel.d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; visual mesh filename=package://drsina_description/models/meshes/topcastlewheel.d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
- link Lwheel_link: mass None -> 0.58215; geometry collision mesh filename=package://drsina_description/models/meshes/robotwheel.dae; visual mesh filename=package://drsina_description/models/meshes/robotwheel.dae
- link RBcastlewheel_link: mass None -> 0.12357; geometry collision mesh filename=package://drsina_description/models/meshes/topcastlewheel.d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; visual mesh filename=package://drsina_description/models/meshes/topcastlewheel.d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
- link RFcastlewheel_link: mass None -> 0.12357; geometry collision mesh filename=package://drsina_description/models/meshes/topcastlewheel.d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; visual mesh filename=package://drsina_description/models/meshes/topcastlewheel.d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
- link Rwheel_link: mass None -> 0.58215; geometry collision mesh filename=package://drsina_description/models/meshes/robotwheel.dae; visual mesh filename=package://drsina_description/models/meshes/robotwheel.dae
- link base_link: mass None -> 28.798; geometry collision box size=0.750 0.750 0.180; visual mesh filename=package://drsina_description/models/meshes/chassis2.dae
- link castlewheel_wheelLBlink: mass None -> 0.194; geometry collision mesh filename=package://drsina_description/models/meshes/castlewheel.dae; visual mesh filename=package://drsina_description/models/meshes/castlewheel.dae
- link castlewheel_wheelLFlink: mass None -> 0.194; geometry collision mesh filename=package://drsina_description/models/meshes/castlewheel.dae; visual mesh filename=package://drsina_description/models/meshes/castlewheel.dae
- link castlewheel_wheelRBlink: mass None -> 0.194; geometry collision mesh filename=package://drsina_description/models/meshes/castlewheel.dae; visual mesh filename=package://drsina_description/models/meshes/castlewheel.dae
- link castlewheel_wheelRFlink: mass None -> 0.194; geometry collision mesh filename=package://drsina_description/models/meshes/castlewheel.dae; visual mesh filename=package://drsina_description/models/meshes/castlewheel.dae
- link emergencyButton_link: mass None -> 0.024; geometry collision cylinder length=0.063 radius=0.015; visual cylinder length=0.063 radius=0.015
- link greenButton_link: mass None -> 0.009; geometry collision cylinder length=0.027 radius=0.015; visual cylinder length=0.027 radius=0.015
- link lidar_link: mass None -> 0.073; geometry collision mesh filename=package://drsina_description/models/meshes/lidarhukuyo.dae; visual mesh filename=package://drsina_description/models/meshes/lidarhukuyo.dae
- link middlecastlewheelLB_link: mass None -> 0.37662; geometry collision mesh filename=package://drsina_description/models/meshes/middlecastkewhee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; visual mesh filename=package://drsina_description/models/meshes/middlecastkewhee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
- link middlecastlewheelLF_link: mass None -> 0.37662; geometry collision mesh filename=package://drsina_description/models/meshes/middlecastkewhee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; visual mesh filename=package://drsina_description/models/meshes/middlecastkewhee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
- link middlecastlewheelRB_link: mass None -> 0.37662; geometry collision mesh filename=package://drsina_description/models/meshes/middlecastkewhee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; visual mesh filename=package://drsina_description/models/meshes/middlecastkewhee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
- link middlecastlewheelRF_link: mass None -> 0.37662; geometry collision mesh filename=package://drsina_description/models/meshes/middlecastkewhee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; visual mesh filename=package://drsina_description/models/meshes/middlecastkewhee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
- link redButton_link: mass None -> 0.009; geometry collision cylinder length=0.027 radius=0.015; visual cylinder length=0.027 radius=0.015
- link redligthL_link: mass None -> 0.013; geometry collision cylinder length=0.035 radius=0.015; visual cylinder length=0.035 radius=0.015
- link redligthR_link: mass None -> 0.013; geometry collision cylinder length=0.035 radius=0.015; visual cylinder length=0.035 radius=0.015
- link yellowligthL_link: mass None -> 0.013; geometry collision cylinder length=0.035 radius=0.015; visual cylinder length=0.035 radius=0.015
- link yellowligthR_link: mass None -> 0.013; geometry collision cylinder length=0.035 radius=0.029; visual cylinder length=0.035 radius=0.015
Joints:
- added joint emergencyButton2_joint: type fixed, parent emergencyButton_link, child emergencyButton2_link, origin xyz=0 0 0 rpy=0 0 0
- added joint joint_name: type fixed, parent base_footprint, child base_link, origin xyz=0.0 0.0 0.0 rpy=0.0 0.0 0.0
- added joint ultrasonic_sensor_back1_joint: type fixed, parent base_link, child ultrasonic_sensor_back1, origin xyz=-0.345 0 0.05 rpy=0 0 3.142
- added joint ultrasonic_sensor_left1_joint: type fixed, parent base_link, child ultrasonic_sensor_left1, origin xyz=0.005 -0.290 0.0 rpy=0 0 -1.570796
- added joint ultrasonic_sensor_right1_joint: type fixed, parent base_link, child ultrasonic_sensor_right1, origin xyz=0.005 0.290 0.0 rpy=0 0 1.570796
- joint lidar_joint: origin xyz=0 0 0 rpy=0 0 0 -> xyz=0.303 -0.006 0.1 rpy=0 0 0

Commit message: Put the differential Pluguin & urdf simplification
new chassis

File: drsina_description/urdf/drsina.urdf (robot description, URDF)
Before this commit: robot DrSina, 28 links, 27 joints
Links:
- removed link base_footprint
- link LBcastlewheel_link: geometry collision box size=0.085 0.105 0.004; visual mesh filename=package://drsina_description/models/meshes/topcastlewheel.d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
- link LFcastlewheel_link: geometry collision box size=0.085 0.105 0.004; visual mesh filename=package://drsina_description/models/meshes/topcastlewheel.d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
- link Lwheel_link: geometry collision cylinder length=0.03 radius=0.075; visual mesh filename=package://drsina_description/models/meshes/robotwheel.dae
- link RBcastlewheel_link: geometry collision box size=0.085 0.105 0.004; visual mesh filename=package://drsina_description/models/meshes/topcastlewheel.d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
- link RFcastlewheel_link: geometry collision box size=0.085 0.105 0.004; visual mesh filename=package://drsina_description/models/meshes/topcastlewheel.d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
- link Rwheel_link: geometry collision cylinder length=0.03 radius=0.075; visual mesh filename=package://drsina_description/models/meshes/robotwheel.dae
- link castlewheel_wheelLBlink: geometry collision cylinder length=0.035 radius=0.05; visual mesh filename=package://drsina_description/models/meshes/castlewheel.dae
- link castlewheel_wheelLFlink: geometry collision cylinder length=0.035 radius=0.05; visual mesh filename=package://drsina_description/models/meshes/castlewheel.dae
- link castlewheel_wheelRBlink: geometry collision cylinder length=0.035 radius=0.05; visual mesh filename=package://drsina_description/models/meshes/castlewheel.dae
- link castlewheel_wheelRFlink: geometry collision cylinder length=0.035 radius=0.05; visual mesh filename=package://drsina_description/models/meshes/castlewheel.dae
Joints:
- removed joint joint_name
- joint roll_jointL: limit effort=100 velocity=100 -> effort=100 velocity=1; origin xyz=-0.0019 0.235 -0.0239 rpy=0 0 0 -> xyz=-0.0019 0.235 -0.0238 rpy=0 0 0
- joint roll_jointR: limit effort=100 velocity=100 -> effort=100 velocity=1; origin xyz=-0.0019 -0.235 -0.0239 rpy=0 0 0 -> xyz=-0.0019 -0.235 -0.0238 rpy=0 0 0
- joint roll_jointcastlewheelLB: limit effort=100 velocity=100 -> effort=1000 velocity=1
- joint roll_jointcastlewheelLF: limit effort=100 velocity=100 -> effort=1000 velocity=1
- joint roll_jointcastlewheelRB: limit effort=100 velocity=100 -> effort=1000 velocity=1
- joint roll_jointcastlewheelRF: limit effort=100 velocity=100 -> effort=1000 velocity=1
- joint roll_jointmiddlecastleLB: limit effort=100 velocity=100 -> effort=1000 velocity=1
- joint roll_jointmiddlecastleLF: limit effort=100 velocity=100 -> effort=1000 velocity=1
- joint roll_jointmiddlecastleRB: limit effort=100 velocity=100 -> effort=1000 velocity=1
- joint roll_jointmiddlecastleRF: limit effort=100 velocity=100 -> effort=1000 velocity=1
