Commit message: The robot's completed URDF

File: hospital_robot/urdf/robot.xacro (robot description, xacro)
@@ -25,5 +25,340 @@
         <color rgba="0.0 0.0  255.0 1.0" />
     </material>
-  <link name="fix">
+    <link name="base_link">
+        <visual>
+            <origin rpy="0.0 0 0" xyz="0 0 0"/>
+            <geometry>
+                <mesh filename="package://hospital_robot/meshes/chassis.dae"/>
+            </geometry>
+            <material name="grey"/>
+        </visual>
+	</link>
+    <link name="Rwheel_link">
+        <visual>
+            <origin rpy="0 0 0" xyz="0.0 0.0 0.0"/>
+            <geometry>
+                <mesh filename="package://hospital_robot/meshes/robotwheel.dae" />
+            </geometry>
+        </visual>
+    </link>
+    <link name="Lwheel_link">
+        <visual>
+            <origin rpy="0 0 3.141592" xyz="0 0 0"/>
+            <geometry>
+                <mesh filename="package://hospital_robot/meshes/robotwheel.dae" />
+            </geometry>
+        </visual>
+    </link>
+    <joint name="roll_jointR" type="continuous">
+    	<parent link="base_link"/>
+    	<child link="Rwheel_link"/>
+        <origin xyz="-0.0019 -0.235 -0.0239" rpy="0 0 0"/>
+        <limit effort="100" velocity="100"/>
+        <axis xyz="0 1 0"/>
+	</joint>
+    <joint name="roll_jointL" type="continuous">
+    	<parent link="base_link"/>
+    	<child link="Lwheel_link"/>
+        <origin xyz="-0.0019 0.235 -0.0239" rpy="0 0 0"/>
+        <limit effort="100" velocity="100"/>
+        <axis xyz="0 1 0"/>
+	</joint>
+<!-- castle Wheel right Backward-->
+    <link name="RBcastlewheel_link">
+        <visual>
+            <origin rpy="0 0 1.570796" xyz="-0.25761 -0.2065 0.027"/>
+            <geometry>
+                <mesh filename="package://hospital_robot/meshes/topcastlewheel.dae" />
+            </geometry>
+        </visual>
+    </link>
+    <joint name="roll_jointcastleRB" type="fixed">
+    	<parent link="base_link"/>
+    	<child link="RBcastlewheel_link"/>
+        <origin xyz="0.0 0 0.0" rpy="0 0 0"/>
+	</joint>
+    <link name="middlecastlewheelRB_link">
+        <visual>
+            <origin xyz="0.0 0 0.0" rpy="0 0 0"/>
+            <!-- <origin rpy="0 0 1.570796" xyz="0 0 0"/> -->
+            <geometry>
+                <mesh filename="package://hospital_robot/meshes/middlecastkewheel.dae" />
+            </geometry>
+        </visual>
+    </link>
+    <joint name="roll_jointmiddlecastleRB" type="continuous">
+    	<parent link="RBcastlewheel_link"/>
+    	<child link="middlecastlewheelRB_link"/>
+        <origin rpy="0 0 1.570796" xyz="-0.25761 -0.2065 0.027"/>
+        <limit effort="100" velocity="100"/>
+        <axis xyz="0 0 1"/>
+	</joint>
+    <link name="castlewheel_wheelRBlink">
+        <visual>
+            <origin xyz="0.0 0 0.0" rpy="0 0 0"/>
+            <geometry>
+                <mesh filename="package://hospital_robot/meshes/castlewheel.dae" />
+            </geometry>
+        </visual>
+    </link>
+    <joint name="roll_jointcastlewheelRB" type="continuous">
+    	<parent link="middlecastlewheelRB_link"/>
+    	<child link="castlewheel_wheelRBlink"/>
+        <!-- <origin rpy="0 0 1.570796" xyz="-0.2890 -0.2065 -0.048"/> -->
+        <origin xyz="0 0.03239 -0.075" rpy="0 0 0"/>
+        <limit effort="100" velocity="100"/>
+        <axis xyz="1 0 0"/>
+	</joint>
+<!--  -->
+<!-- castle Wheel right Forward-->
+    <link name="RFcastlewheel_link">
+        <visual>
+            <origin rpy="0 0 1.570796" xyz="0.25761 -0.2065 0.027"/>
+            <geometry>
+                <mesh filename="package://hospital_robot/meshes/topcastlewheel.dae" />
+            </geometry>
+        </visual>
+    </link>
+    <joint name="roll_jointcastleRF" type="fixed">
+    	<parent link="base_link"/>
+    	<child link="RFcastlewheel_link"/>
+        <origin xyz="0.0 0 0.0" rpy="0 0 0"/>
+	</joint>
+    <link name="middlecastlewheelRF_link">
+        <visual>
+            <origin xyz="0.0 0 0.0" rpy="0 0 0"/>
+            <geometry>
+                <mesh filename="package://hospital_robot/meshes/middlecastkewheel.dae" />
+            </geometry>
+        </visual>
+    </link>
+    <joint name="roll_jointmiddlecastleRF" type="continuous">
+    	<parent link="RFcastlewheel_link"/>
+    	<child link="middlecastlewheelRF_link"/>
+        <origin rpy="0 0 1.570796" xyz="0.25761 -0.2065 0.027"/>
+        <limit effort="100" velocity="100"/>
+        <axis xyz="0 0 1"/>
+	</joint>
+    <link name="castlewheel_wheelRFlink">
+        <visual>
+            <origin xyz="0.0 0 0.0" rpy="0 0 0"/>
+            <geometry>
+                <mesh filename="package://hospital_robot/meshes/castlewheel.dae" />
+            </geometry>
+        </visual>
+    </link>
+    <joint name="roll_jointcastlewheelRF" type="continuous">
+    	<parent link="middlecastlewheelRF_link"/>
+    	<child link="castlewheel_wheelRFlink"/>
+        <!-- <origin rpy="0 0 1.570796" xyz="0.2240 -0.2065 -0.048"/> -->
+        <origin xyz="0 0.03239 -0.075" rpy="0 0 0"/>
+        <limit effort="100" velocity="100"/>
+        <axis xyz="1 0 0"/>
+	</joint>
+<!--  -->
+<!-- castle Wheel Left Forward-->
+    <link name="LFcastlewheel_link">
+        <visual>
+            <origin rpy="0 0 1.570796" xyz="0.25761 0.2065 0.027"/>
+            <geometry>
+                <mesh filename="package://hospital_robot/meshes/topcastlewheel.dae" />
+            </geometry>
+        </visual>
+    </link>
+    <joint name="roll_jointcastleLF" type="fixed">
+    	<parent link="base_link"/>
+    	<child link="LFcastlewheel_link"/>
+        <origin xyz="0.0 0 0.0" rpy="0 0 0"/>
+	</joint>
+    <link name="middlecastlewheelLF_link">
+        <visual>
+            <origin xyz="0.0 0 0.0" rpy="0 0 0"/>
+            <geometry>
+                <mesh filename="package://hospital_robot/meshes/middlecastkewheel.dae" />
+            </geometry>
+        </visual>
+    </link>
+    <joint name="roll_jointmiddlecastleLF" type="continuous">
+    	<parent link="LFcastlewheel_link"/>
+    	<child link="middlecastlewheelLF_link"/>
+        <origin rpy="0 0 1.570796" xyz="0.25761 0.2065 0.027"/>
+        <limit effort="100" velocity="100"/>
+        <axis xyz="0 0 1"/>
+	</joint>
+    <link name="castlewheel_wheelLFlink">
+        <visual>
+            <origin xyz="0.0 0 0.0" rpy="0 0 0"/>
+            <geometry>
+                <mesh filename="package://hospital_robot/meshes/castlewheel.dae" />
+            </geometry>
+        </visual>
+    </link>
+    <joint name="roll_jointcastlewheelLF" type="continuous">
+    	<parent link="middlecastlewheelLF_link"/>
+    	<child link="castlewheel_wheelLFlink"/>
+        <origin  xyz="0 0.03239 -0.075" rpy="0 0 0"/>
+        <limit effort="100" velocity="100"/>
+        <axis xyz="1 0 0"/>
+	</joint>
+<!--  -->
+<!-- castle Wheel Left Backward-->
+    <link name="LBcastlewheel_link">
+        <visual>
+            <origin rpy="0 0 1.570796" xyz="-0.25761 0.2065 0.027"/>
+            <geometry>
+                <mesh filename="package://hospital_robot/meshes/topcastlewheel.dae" />
+            </geometry>
+        </visual>
+    </link>
+    <joint name="roll_jointcastleLB" type="fixed">
+    	<parent link="base_link"/>
+    	<child link="LBcastlewheel_link"/>
+        <origin xyz="0.0 0 0.0" rpy="0 0 0"/>
+	</joint>
+    <link name="middlecastlewheelLB_link">
+        <visual>
+            <origin xyz="0.0 0 0.0" rpy="0 0 0"/>
+            <geometry>
+                <mesh filename="package://hospital_robot/meshes/middlecastkewheel.dae" />
+            </geometry>
+        </visual>
+    </link>
+    <joint name="roll_jointmiddlecastleLB" type="continuous">
+    	<parent link="LBcastlewheel_link"/>
+    	<child link="middlecastlewheelLB_link"/>
+        <origin rpy="0 0 1.570796" xyz="-0.25761 0.2065 0.027"/>
+        <limit effort="100" velocity="100"/>
+        <axis xyz="0 0 1"/>
+	</joint>
+    <link name="castlewheel_wheelLBlink">
+        <visual>
+            <origin xyz="0.0 0 0.0" rpy="0 0 0"/>
+            <geometry>
+                <mesh filename="package://hospital_robot/meshes/castlewheel.dae" />
+            </geometry>
+        </visual>
+    </link>
+    <joint name="roll_jointcastlewheelLB" type="continuous">
+    	<parent link="middlecastlewheelLB_link"/>
+    	<child link="castlewheel_wheelLBlink"/>
+        <origin xyz="0 0.03239 -0.075" rpy="0 0 0"/>
+        <limit effort="100" velocity="100"/>
+        <axis xyz="1 0 0"/>
+	</joint>
+<!--  -->
+<!-- Light indicator -->
+    <link name="emergencyButton_link">
+        <visual>
+            <origin rpy="0 -1.570796 0" xyz="-0.360 0 0"/>
+            <geometry>
+                <mesh filename="package://hospital_robot/meshes/emergencyButton.dae" />
+            </geometry>
+        </visual>
+    </link>
+    <joint name="emergencyButton_joint" type="fixed">
+    	<parent link="base_link"/>
+    	<child link="emergencyButton_link"/>
+        <origin xyz="0 0 0" rpy="0 0 0"/>
+	</joint>
+    <link name="yellowligthR_link">
+        <visual>
+            <origin rpy="0 -1.570796 0" xyz="-0.365 0.158 0"/>
+            <geometry>
+                <mesh filename="package://hospital_robot/meshes/lightback.dae" />
+            </geometry>
+        </visual>
+    </link>
+    <joint name="yellowligthR_joint" type="fixed">
+    	<parent link="base_link"/>
+    	<child link="yellowligthR_link"/>
+        <origin xyz="0 0 0" rpy="0 0 0"/>
+	</joint>
+    <link name="yellowligthL_link">
+        <visual>
+            <origin rpy="0 -1.570796 0" xyz="-0.365 -0.158 0"/>
+            <geometry>
+                <mesh filename="package://hospital_robot/meshes/lightback.dae" />
+            </geometry>
+        </visual>
+    </link>
+    <joint name="yellowligthL_joint" type="fixed">
+    	<parent link="base_link"/>
+    	<child link="yellowligthL_link"/>
+        <origin xyz="0 0 0" rpy="0 0 0"/>
+	</joint>
+    <link name="redligthR_link">
+        <visual>
+            <origin rpy="0 -1.570796 0" xyz="-0.365 0.095 0"/>
+            <geometry>
+                <mesh filename="package://hospital_robot/meshes/lightbackRed.dae" />
+            </geometry>
+        </visual>
+    </link>
+    <joint name="redligthR_joint" type="fixed">
+    	<parent link="base_link"/>
+    	<child link="redligthR_link"/>
+        <origin xyz="0 0 0" rpy="0 0 0"/>
+	</joint>
+    <link name="redligthL_link">
+        <visual>
+            <origin rpy="0 -1.570796 0" xyz="-0.365 -0.095 0"/>
+            <geometry>
+                <mesh filename="package://hospital_robot/meshes/lightbackRed.dae" />
+            </geometry>
+        </visual>
+    </link>
+    <joint name="redligthL_joint" type="fixed">
+    	<parent link="base_link"/>
+    	<child link="redligthL_link"/>
+        <origin xyz="0 0 0" rpy="0 0 0"/>
+	</joint>
+<!--  -->
+<!-- green button -->
+    <link name="greenButton_link">
+        <visual>
+            <origin rpy="0 0 0" xyz="0.298 0.1001 0.075"/>
+            <geometry>
+                <mesh filename="package://hospital_robot/meshes/buttongreen.dae" />
+            </geometry>
+        </visual>
+    </link>
+    <joint name="greenButton_joint" type="fixed">
+    	<parent link="base_link"/>
+    	<child link="greenButton_link"/>
+        <origin xyz="0 0 0" rpy="0 0 0"/>
+	</joint>
+<!--  -->
+<!-- red Button -->
+    <link name="redButton_link">
+        <visual>
+            <origin rpy="0 0 0" xyz="0.298 -0.1001 0.075"/>
+            <geometry>
+                <mesh filename="package://hospital_robot/meshes/buttonred.dae" />
+            </geometry>
+        </visual>
+    </link>
+    <joint name="redButton_joint" type="fixed">
+    	<parent link="base_link"/>
+    	<child link="redButton_link"/>
+        <origin xyz="0 0 0" rpy="0 0 0"/>
+	</joint>
+<!--  -->
+<!-- lidar  -->
+    <link name="lidar_link">
+        <visual>
+            <origin rpy="0 0 0" xyz="0.303 -0.006 0.1"/>
+            <geometry>
+                <mesh filename="package://hospital_robot/meshes/lidar.dae" />
+            </geometry>
+        </visual>
+    </link>
+    <joint name="lidar_joint" type="fixed">
+    	<parent link="base_link"/>
+    	<child link="lidar_link"/>
+        <origin xyz="0 0 0" rpy="0 0 0"/>
+	</joint>
+<!--  -->
+<!-- base armoire link  -->
+    <link name="fix">
      <pose>0 0 0 0 0 0</pose>
         <inertial>
@@ -39,5 +374,5 @@
             </inertial>
         <collision>
-            <origin xyz="0 0 0.3" rpy="1.57 0 0" />
+            <origin xyz="0 0 0" rpy="1.57 0 0" />
             <geometry>
                 <mesh filename="package://hospital_robot/meshes/fix.stl" />
@@ -45,5 +380,5 @@
         </collision>
         <visual>
-            <origin xyz="0 0 0.3" rpy="1.57 0 0" />
+            <origin xyz="0 0 0" rpy="1.57 0 0" />
             <geometry>
                 <mesh
@@ -53,4 +388,11 @@
         </visual>
     </link>
+    <joint name="principle_joint" type="fixed">
+        <origin xyz="-0.3 0 0.19" rpy="0 0 0" />
+    	<parent link="base_link"/>
+    	<child link="fix"/>
+        <origin xyz="0 0 0" rpy="0 0 0"/>
+	</joint>
+<!--  -->
     <link name="lampe">
      <pose>0 0 0 0 0 0</pose>
@@ -82,5 +424,5 @@
     </link>
   <joint name="lampe_joint" type="fixed">
-    <origin xyz="0.2 -0.05 1.31" rpy="0 0 0" />
+    <origin xyz="0.2 -0.05 1.01" rpy="0 0 0" />
     <parent link="fix" />
     <child link="lampe" />
@@ -105,5 +447,5 @@
     </link>
     <joint name="sep1_joint" type="fixed">
-    <origin xyz="0.345 0.21 0.31" rpy="0 0 0" />
+    <origin xyz="0.345 0.21 0.01" rpy="0 0 0" />
     <parent link="fix" />
     <child link="sep1" />
@@ -128,5 +470,5 @@
     </link>
     <joint name="sep2_joint" type="fixed">
-    <origin xyz="0.25 0.15 0.31" rpy="0 0 0" />
+    <origin xyz="0.25 0.15 0.01" rpy="0 0 0" />
     <parent link="fix" />
     <child link="sep2" />
@@ -151,5 +493,5 @@
     </link>
     <joint name="sep1.2_joint" type="fixed">
-    <origin xyz="0.07 -0.21 0.31" rpy="0 0 0" />
+    <origin xyz="0.07 -0.21 0.01" rpy="0 0 0" />
     <parent link="fix" />
     <child link="sep1.2" />
@@ -174,5 +516,5 @@
     </link>
     <joint name="sep2.2_joint" type="fixed">
-    <origin xyz="0.255 -0.28 0.31" rpy="0 0 0" />
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