Commit message: Add dae files and joint publisher with correct limit prismatic

File: hospital_robot/urdf/robot.xacro (robot description, xacro)
@@ -26,5 +26,4 @@
     </material>
   <link name="fix">
-     <pose>0 0 0 0 0 0</pose>
         <inertial>
             <origin xyz="0 0 0" rpy="0 0 0" />
@@ -41,5 +40,5 @@
             <origin xyz="0 0 0.3" rpy="1.57 0 0" />
             <geometry>
-                <mesh filename="package://hospital_robot/meshes/fix.stl" />
+                <mesh filename="package://hospital_robot/meshes/fix.dae" />
             </geometry>
         </collision>
@@ -48,11 +47,9 @@
             <geometry>
                 <mesh
-                filename="package://hospital_robot/meshes/fix.stl" />
-            </geometry>
-            <material name="silver"/>
+                filename="package://hospital_robot/meshes/fix.dae" />
+            </geometry>
         </visual>
     </link>
     <link name="lampe">
-     <pose>0 0 0 0 0 0</pose>
         <inertial>
             <origin xyz="0 0 0" rpy="0 0 0" />
@@ -69,14 +66,13 @@
             <origin xyz="0 0 0" rpy="0 0 1.57" />
             <geometry>
-                <mesh filename="package://hospital_robot/meshes/lampe.stl" />
-            </geometry>
-        </collision>
-        <visual>
-            <origin xyz="0 0 0" rpy="0 0 1.57" />
-            <geometry>
-                <mesh
-                filename="package://hospital_robot/meshes/lampe.stl" />
-            </geometry>
-            <material name="red"/>
+                <mesh filename="package://hospital_robot/meshes/lampe.dae" />
+            </geometry>
+        </collision>
+        <visual>
+            <origin xyz="0 0 0" rpy="0 0 1.57" />
+            <geometry>
+                <mesh
+                filename="package://hospital_robot/meshes/lampe.dae" />
+            </geometry>
         </visual>
     </link>
@@ -88,9 +84,8 @@
   </joint>
   <link name="sep1">
-     <pose>0 0 0 0 0 0</pose>
         <collision>
             <origin xyz="0 0 0" rpy="0 0 3.14" />
             <geometry>
-                <mesh filename="package://hospital_robot/meshes/sep_complexe.stl" />
+                <mesh filename="package://hospital_robot/meshes/sepcomplex.dae" />
             </geometry>
         </collision>
@@ -99,7 +94,6 @@
             <geometry>
                 <mesh
-                filename="package://hospital_robot/meshes/sep_complexe.stl" />
-            </geometry>
-            <material name="cyan"/>
+                filename="package://hospital_robot/meshes/sepcomplex.dae" />
+            </geometry>
         </visual>
     </link>
@@ -111,18 +105,16 @@
   </joint>
   <link name="sep2">
-     <pose>0 0 0 0 0 0</pose>
-        <collision>
-            <origin xyz="0 0 0" rpy="0 0 1.57" />
-            <geometry>
-                <mesh filename="package://hospital_robot/meshes/sep_simple.stl" />
-            </geometry>
-        </collision>
-        <visual>
-            <origin xyz="0 0 0" rpy="0 0 1.57" />
-            <geometry>
-                <mesh
-                filename="package://hospital_robot/meshes/sep_simple.stl" />
-            </geometry>
-            <material name="cyan"/>
+        <collision>
+            <origin xyz="0 0 0" rpy="0 0 1.57" />
+            <geometry>
+                <mesh filename="package://hospital_robot/meshes/sep_simple.dae" />
+            </geometry>
+        </collision>
+        <visual>
+            <origin xyz="0 0 0" rpy="0 0 1.57" />
+            <geometry>
+                <mesh
+                filename="package://hospital_robot/meshes/sep_simple.dae" />
+            </geometry>
         </visual>
     </link>
@@ -134,18 +126,16 @@
   </joint>
   <link name="sep1.2">
-     <pose>0 0 0 0 0 0</pose>
-        <collision>
-            <origin xyz="0 0 0" rpy="0 0 0" />
-            <geometry>
-                <mesh filename="package://hospital_robot/meshes/sep_complexe.stl" />
-            </geometry>
-        </collision>
-        <visual>
-            <origin xyz="0 0 0" rpy="0 0 0" />
-            <geometry>
-                <mesh
-                filename="package://hospital_robot/meshes/sep_complexe.stl" />
-            </geometry>
-            <material name="cyan"/>
+        <collision>
+            <origin xyz="0 0 0" rpy="0 0 0" />
+            <geometry>
+                <mesh filename="package://hospital_robot/meshes/sepcomplex.dae" />
+            </geometry>
+        </collision>
+        <visual>
+            <origin xyz="0 0 0" rpy="0 0 0" />
+            <geometry>
+                <mesh
+                filename="package://hospital_robot/meshes/sepcomplex.dae" />
+            </geometry>
         </visual>
     </link>
@@ -157,18 +147,16 @@
   </joint>
   <link name="sep2.2">
-     <pose>0 0 0 0 0 0</pose>
-        <collision>
-            <origin xyz="0 0 0" rpy="0 0 1.57" />
-            <geometry>
-                <mesh filename="package://hospital_robot/meshes/sep_simple.stl" />
-            </geometry>
-        </collision>
-        <visual>
-            <origin xyz="0 0 0" rpy="0 0 1.57" />
-            <geometry>
-                <mesh
-                filename="package://hospital_robot/meshes/sep_simple.stl" />
-            </geometry>
-            <material name="cyan"/>
+        <collision>
+            <origin xyz="0 0 0" rpy="0 0 1.57" />
+            <geometry>
+                <mesh filename="package://hospital_robot/meshes/sep_simple.dae" />
+            </geometry>
+        </collision>
+        <visual>
+            <origin xyz="0 0 0" rpy="0 0 1.57" />
+            <geometry>
+                <mesh
+                filename="package://hospital_robot/meshes/sep_simple.dae" />
+            </geometry>
         </visual>
     </link>
@@ -180,5 +168,4 @@
   </joint>
   <link name="montechargeL">
-     <pose>0 0 0 0 0 0</pose>
         <collision>
             <origin xyz="0 0 0" rpy="0 0 0" />
@@ -201,8 +188,7 @@
     <child link="montechargeL" />
     <axis xyz="0 0 1" />
-    <limit effort="1000.0" lower="0.35" upper="1.0" velocity="0.5"/>
+    <limit effort="1000.0" lower="0.2" upper="0.89" velocity="0.5"/>
   </joint>
   <link name="montechargeR">
-     <pose>0 0 0 0 0 0</pose>
         <collision>
             <origin xyz="0 0 0" rpy="3.14 0 0" />
@@ -225,19 +211,18 @@
     <child link="montechargeR" />
     <axis xyz="0 0 1" />
-    <limit effort="1000.0" lower="0.35" upper="1.0" velocity="0.5"/>
+    <limit effort="1000.0" lower="0.2" upper="0.89" velocity="0.5"/>
   </joint>
   <link name="kjarL">
-     <pose>0 0 0 0 0 0</pose>
-        <collision>
-            <origin xyz="0 0 0" rpy="0 0 1.57" />
-            <geometry>
-                <mesh filename="package://hospital_robot/meshes/kjar.stl" />
-            </geometry>
-        </collision>
-        <visual>
-            <origin xyz="0 0 0" rpy="0 0 1.57" />
-            <geometry>
-                <mesh
-                filename="package://hospital_robot/meshes/kjar.stl" />
+        <collision>
+            <origin xyz="0 0 0" rpy="0 0 1.57" />
+            <geometry>
+                <mesh filename="package://hospital_robot/meshes/kjar.dae" />
+            </geometry>
+        </collision>
+        <visual>
+            <origin xyz="0 0 0" rpy="0 0 1.57" />
+            <geometry>
+                <mesh
+                filename="package://hospital_robot/meshes/kjar.dae" />
             </geometry>
             <material name="black"/>
@@ -245,16 +230,15 @@
     </link>
     <joint name="kjar_joint" type="prismatic">
-    <origin xyz=" 0.51 -0.15 1.23" rpy="0 0 0" />
+    <origin xyz=" 0.51 -0.15 1.237" rpy="0 0 0" />
     <parent link="fix" />
     <child link="kjarL" />
     <axis xyz="0 1 0" />
-    <limit effort="100.0" lower="0.1" upper="0.3" velocity="0.5"/>
+    <limit effort="100.0" lower="0.001" upper="0.4" velocity="0.5"/>
   </joint>
   <link name="kjarR">
-     <pose>0 0 0 0 0 0</pose>
         <collision>
             <origin xyz="0 0 0" rpy="0 0 -1.57" />
             <geometry>
-                <mesh filename="package://hospital_robot/meshes/kjar.stl" />
+                <mesh filename="package://hospital_robot/meshes/kjar.dae" />
             </geometry>
         </collision>
@@ -263,5 +247,5 @@
             <geometry>
                 <mesh
-                filename="package://hospital_robot/meshes/kjar.stl" />
+                filename="package://hospital_robot/meshes/kjar.dae" />
             </geometry>
             <material name="black"/>
@@ -269,12 +253,11 @@
     </link>
     <joint name="kjarR_joint" type="prismatic">
-    <origin xyz=" 0.40 -0.24 1.23" rpy="0 0 0" />
+    <origin xyz=" 0.3965 -0.25 1.239" rpy="0 0 0" />
     <parent link="fix" />
     <child link="kjarR" />
     <axis xyz="0 1 0" />
-    <limit effort="100.0" lower="0.1" upper="0.3" velocity="0.5"/>
+    <limit effort="100.0" lower="0.001" upper="0.4" velocity="0.5"/>
   </joint>
   <link name="plat">
-     <pose>0 0 0 0 0 0</pose>
         <collision>
             <origin xyz="0 0 0" rpy="3.14 0 1.57" />
@@ -293,34 +276,31 @@
     </link>
     <joint name="plat_joint" type="fixed">
-    <origin xyz="0.06 0.14 0.06 " rpy="0 0 0" />
-    <parent link="montechargeR" />
+    <origin xyz="0.06 0.05 0.06 " rpy="0 0 0" />
+    <parent link="montechargeL" />
     <child link="plat" />
     <axis xyz="0 0 0" />
   </joint>
   <link name="bottle">
-     <pose>0 0 0 0 0 0</pose>
-        <collision>
-            <origin xyz="0 0 0" rpy="0 0 0" />
-            <geometry>
-                <mesh filename="package://hospital_robot/meshes/bottle.stl" />
-            </geometry>
-        </collision>
-        <visual>
-            <origin xyz="0 0 0" rpy="0 0 0" />
-            <geometry>
-                <mesh
-                filename="package://hospital_robot/meshes/bottle.stl" />
-            </geometry>
-            <material name="blue"/>
+        <collision>
+            <origin xyz="0 0 0" rpy="0 0 0" />
+            <geometry>
+                <mesh filename="package://hospital_robot/meshes/bottle.dae" />
+            </geometry>
+        </collision>
+        <visual>
+            <origin xyz="0 0 0" rpy="0 0 0" />
+            <geometry>
+                <mesh
+                filename="package://hospital_robot/meshes/bottle.dae" />
+            </geometry>
         </visual>
     </link>
     <joint name="bottle_joint" type="fixed">
-    <origin xyz="0.23 0.15 0 " rpy="0 0 0" />
-    <parent link="montechargeR" />
+    <origin xyz="0.23 0.05 0 " rpy="0 0 0" />
+    <parent link="montechargeL" />
     <child link="bottle" />
     <axis xyz="0 0 0" />
   </joint>
   <link name="porteL">
-     <pose>0 0 0 0 0 0</pose>
         <collision>
             <origin xyz="0 0 0" rpy="0 -1.57 1.57" />
@@ -345,5 +325,4 @@
   </joint>
   <link name="porteR">
-     <pose>0 0 0 0 0 0</pose>
         <collision>
             <origin xyz="0 0 0" rpy="0 -1.57 1.57" />
@@ -368,5 +347,4 @@
   </joint>
   <link name="yedL">
-     <pose>0 0 0 0 0 0</pose>
         <collision>
             <origin xyz="0 0 0" rpy="0 0 0" />
@@ -391,5 +369,4 @@
   </joint>
   <link name="yedR">
-     <pose>0 0 0 0 0 0</pose>
         <collision>
             <origin xyz="0 0 0" rpy="0 0 3.14" />
@@ -414,5 +391,4 @@
   </joint>
   <link name="yedF">
-     <pose>0 0 0 0 0 0</pose>
         <collision>
             <origin xyz="0 0 0" rpy="0 0 -1.57" />
@@ -436,56 +412,9 @@
     <axis xyz="0 0 0" />
   </joint>
-  <link name="gjouraL">
-     <pose>0 0 0 0 0 0</pose>
-        <collision>
-            <origin xyz="0 0 0" rpy="0 0 1.57" />
-            <geometry>
-                <mesh filename="package://hospital_robot/meshes/9joura.stl" />
-            </geometry>
-        </collision>
-        <visual>
-            <origin xyz="0 0 0" rpy="0 0 1.57" />
-            <geometry>
-                <mesh
-                filename="package://hospital_robot/meshes/9joura.stl" />
-            </geometry>
-            <material name="black"/>
-        </visual>
-    </link>
-    <joint name="kjouraL_joint" type="fixed">
-    <origin xyz="0.50 0.04 0.44  " rpy="0 0 0" />
-    <parent link="fix" />
-    <child link="gjouraL" />
-    <axis xyz="0 0 0" />
-  </joint>
-  <link name="gjouraR">
-     <pose>0 0 0 0 0 0</pose>
-        <collision>
-            <origin xyz="0 0 0" rpy="0 0 -1.57" />
-            <geometry>
-                <mesh filename="package://hospital_robot/meshes/9joura.stl" />
-            </geometry>
-        </collision>
-        <visual>
-            <origin xyz="0 0 0" rpy="0 0 -1.57" />
-            <geometry>
-                <mesh
-                filename="package://hospital_robot/meshes/9joura.stl" />
-            </geometry>
-            <material name="black"/>
-        </visual>
-    </link>
-    <joint name="kjouraR_joint" type="fixed">
-    <origin xyz="0.40 -0.04 0.44  " rpy="0 0 0" />
-    <parent link="fix" />
-    <child link="gjouraR" />
-    <axis xyz="0 0 0" />
-  </joint>
   <link name="liaison">
-     <pose>0 0 0 0 0 0</pose>
         <collision>
             <origin xyz="0 0 0" rpy="1.57 0 0" />
             <geometry>
-                <mesh filename="package://hospital_robot/meshes/liaison.stl" />
+                <mesh filename="package://hospital_robot/meshes/liaison.dae" />
             </geometry>
         </collision>
@@ -494,7 +423,6 @@
             <geometry>
                 <mesh
-                filename="package://hospital_robot/meshes/liaison.stl" />
-            </geometry>
-            <material name="cyan"/>
+                filename="package://hospital_robot/meshes/liaison.dae" />
+            </geometry>
         </visual>
     </link>
