Commit message: trying diff plugin from gazebo

File: drsina/drsina_description/urdf/drsina.urdf (robot description, URDF)
Before this commit: robot DrSina, 27 links, 26 joints
Links:
- removed link base_footprint
- added link emergencyButton2_link, mass 0.024; collision cylinder length=0.007 radius=0.025; visual cylinder length=0.007 radius=0.025
- link base_link: geometry collision box size=0.750 0.750 0.180; visual mesh filename=package://drsina_description/models/meshes/chassis2.dae
- link emergencyButton_link: geometry collision cylinder length=0.063 radius=0.015; visual cylinder length=0.063 radius=0.015
- link greenButton_link: geometry collision cylinder length=0.027 radius=0.015; visual cylinder length=0.027 radius=0.015
- link lidar_link: geometry collision mesh filename=package://drsina_description/models/meshes/lidarhukuyo.dae; visual mesh filename=package://drsina_description/models/meshes/lidarhukuyo.dae
- link redButton_link: geometry collision cylinder length=0.027 radius=0.015; visual cylinder length=0.027 radius=0.015
- link redligthL_link: geometry collision cylinder length=0.035 radius=0.015; visual cylinder length=0.035 radius=0.015
- link redligthR_link: geometry collision cylinder length=0.035 radius=0.015; visual cylinder length=0.035 radius=0.015
- link yellowligthL_link: geometry collision cylinder length=0.035 radius=0.015; visual cylinder length=0.035 radius=0.015
- link yellowligthR_link: geometry collision cylinder length=0.035 radius=0.029; visual cylinder length=0.035 radius=0.015
Joints:
- removed joint joint_name
- added joint emergencyButton2_joint: type fixed, parent emergencyButton_link, child emergencyButton2_link, origin xyz=0 0 0 rpy=0 0 0

Commit message: robot well and running

File: drsina/drsina_description/urdf/drsina.urdf (robot description, URDF)
Before this commit: robot DrSina, 27 links, 26 joints
Links:
- added link base_footprint
Joints:
- added joint base_joint: type fixed, parent base_footprint, child base_link, origin xyz=0.0 0.0 0.0 rpy=0.0 0.0 0.0
- joint roll_jointcastlewheelLF: origin xyz=0 0.03239 -0.075 rpy=0 0 0 -> xyz=0 0.03239 -0.076 rpy=0 0 0
- joint roll_jointcastlewheelRF: origin xyz=0 0.03239 -0.075 rpy=0 0 0 -> xyz=0 0.03239 -0.076 rpy=0 0 0

Commit message: Take Master Drsina And Add Camera to the Base

File: drsina/drsina_description/urdf/drsina.urdf (robot description, URDF)
Before this commit: robot DrSina, 27 links, 26 joints
Links:
- added link base_footprint
- added link camera_link, mass 1e-5; collision box size=0.01 0.05 0.05; visual box size=0.01 0.05 0.05
- added link camera_offset; visual box size=0.01 0.01 0.01
Joints:
- added joint base_joint: type fixed, parent base_footprint, child base_link, origin xyz=0.0 0.0 0.0 rpy=0.0 0.0 0.0
- added joint camera_joint: type fixed, parent base_link, child camera_link, origin xyz=0.372 0 0 rpy=0 0 0
- added joint camera_offset_joint: type fixed, parent camera_link, child camera_offset, origin xyz=0.01 0 0 rpy=0 0 0
- joint roll_jointcastlewheelLF: origin xyz=0 0.03239 -0.075 rpy=0 0 0 -> xyz=0 0.03239 -0.076 rpy=0 0 0
- joint roll_jointcastlewheelRF: origin xyz=0 0.03239 -0.075 rpy=0 0 0 -> xyz=0 0.03239 -0.076 rpy=0 0 0

Commit message: upper base of the robot

File: drsina/drsina_description/urdf/drsina.urdf (robot description, URDF)
Before this commit: robot DrSina, 28 links, 27 joints
Links:
- added link camera_depth_frame
- added link camera_depth_optical_frame
- added link camera_rgb_frame
- added link camera_rgb_optical_frame
- added link kinect_link, mass 0.564; collision box size=0.07271 0.27794 0.073; visual mesh filename=package://penguin_description/models/meshes/kinect.dae
- added link upper_link, mass 2.0; collision box size=0.7 0.7 1.12; visual mesh filename=package://drsina_description/models/meshes/fou95.dae
Joints:
- added joint camera_depth_joint: type fixed, parent camera_rgb_frame, child camera_depth_frame, origin xyz=0 0.0 0 rpy=0 0 0
- added joint camera_depth_optical_joint: type fixed, parent camera_depth_frame, child camera_depth_optical_frame, origin xyz=0 0 0 rpy=-1.5707 0 -1.5707
- added joint camera_rgb_joint: type fixed, parent base_link, child camera_rgb_frame, origin xyz=0.25 0.0 1.15 rpy=0 0 0
- added joint camera_rgb_optical_joint: type fixed, parent camera_rgb_frame, child camera_rgb_optical_frame, origin xyz=0 0 0 rpy=-1.5707 0 -1.5707
- added joint kinect_base_joint: type fixed, parent camera_rgb_frame, child kinect_link, origin xyz=0 0 0 rpy=0.0 0.0 0.0
- added joint top_joint: type fixed, parent base_link, child upper_link, origin xyz=0.0 0.0 0.02 rpy=0.0 0.0 -1.5707

Commit message: added the hospital map to the package drsina

File: drsina/drsina_description/urdf/drsina.urdf (robot description, URDF)
Before this commit: robot DrSina, 31 links, 30 joints
Links:
- removed link camera_link
- removed link camera_offset
- removed link upper_part_link
- added link camera_depth_frame
- added link camera_depth_optical_frame
- added link camera_rgb_frame
- added link camera_rgb_optical_frame
- added link kinect_link, mass 0.564; collision box size=0.07271 0.27794 0.073; visual mesh filename=package://penguin_description/models/meshes/kinect.dae
- added link upper_link, mass 2.0; collision box size=0.7 0.7 1.12; visual mesh filename=package://drsina_description/models/meshes/fou95.dae
Joints:
- removed joint camera_joint
- removed joint camera_offset_joint
- removed joint upper_part_joint
- added joint camera_depth_joint: type fixed, parent camera_rgb_frame, child camera_depth_frame, origin xyz=0 0.0 0 rpy=0 0 0
- added joint camera_depth_optical_joint: type fixed, parent camera_depth_frame, child camera_depth_optical_frame, origin xyz=0 0 0 rpy=-1.5707 0 -1.5707
- added joint camera_rgb_joint: type fixed, parent base_link, child camera_rgb_frame, origin xyz=0.25 0.0 1.15 rpy=0 0 0
- added joint camera_rgb_optical_joint: type fixed, parent camera_rgb_frame, child camera_rgb_optical_frame, origin xyz=0 0 0 rpy=-1.5707 0 -1.5707
- added joint kinect_base_joint: type fixed, parent camera_rgb_frame, child kinect_link, origin xyz=0 0 0 rpy=0.0 0.0 0.0
- added joint top_joint: type fixed, parent base_link, child upper_link, origin xyz=0.0 0.0 0.02 rpy=0.0 0.0 -1.5707
